Commit message: fix laser noise? bug

File: urdf/turtlebot3_waffle_pi.gazebo.xacro (robot description, xacro)
@@ -106,5 +106,5 @@
     <sensor type="ray" name="lds_lfcd_sensor">
       <pose>0 0 0 0 0 0</pose>
-      <visualize>$(arg laser_visual)</visualize>
+      <visualize>true</visualize>
       <update_rate>5</update_rate>
       <ray>
@@ -119,5 +119,5 @@
         <range>
           <min>0.120</min>
-          <max>3.5</max>
+          <max>30</max>
           <resolution>0.015</resolution>
         </range>

File: urdf/turtlebot3_waffle_pi_with_d435.urdf.xacro (robot description, xacro)
@@ -137,5 +137,5 @@
     <parent link="base_link"/>
     <child link="base_scan"/>
-    <origin xyz="-0.064 0 0.122" rpy="0 0 0"/>
+    <origin xyz="-0.064 0 1" rpy="0 0 0"/>
   </joint>
   <link name="base_scan">
