Commit message: まだ動作せず｡RGBカメラ用の記述を削除｡ takuya@takuya-blade:~$ roslaunch turtlebot3_navigation turtlebot3_navigation_laser_limit.launch ... logging to /home/takuya/.ros/log/2019eb2c-4054-11eb-b925-b827eb5b1dad/roslaunch-takuya-blade-25824.log Checking log directory for disk usage. This may take a while. Press Ctrl-C to interrupt Done checking log file disk usage. Usage is <1GB.
xacro: in-order processing became default in ROS Melodic. You can drop the option.
started roslaunch server http://takuya-blade.local:42791/

SUMMARY
========

PARAMETERS
 * /amcl/base_frame_id: base_footprint
 * /amcl/gui_publish_rate: 50.0
 * /amcl/initial_pose_a: 0.0
 * /amcl/initial_pose_x: 0.0
 * /amcl/initial_pose_y: 0.0
 * /amcl/kld_err: 0.02
 * /amcl/laser_lambda_short: 0.1
 * /amcl/laser_likelihood_max_dist: 2.0
 * /amcl/laser_max_beams: 180
 * /amcl/laser_max_range: 3.5
 * /amcl/laser_min_range: 0.3
 * /amcl/laser_model_type: likelihood_field
 * /amcl/laser_sigma_hit: 0.2
 * /amcl/laser_z_hit: 0.5
 * /amcl/laser_z_max: 0.05
 * /amcl/laser_z_rand: 0.5
 * /amcl/laser_z_short: 0.05
 * /amcl/max_particles: 3000
 * /amcl/min_particles: 500
 * /amcl/odom_alpha1: 0.1
 * /amcl/odom_alpha2: 0.1
 * /amcl/odom_alpha3: 0.1
 * /amcl/odom_alpha4: 0.1
 * /amcl/odom_frame_id: odom
 * /amcl/odom_model_type: diff
 * /amcl/recovery_alpha_fast: 0.0
 * /amcl/recovery_alpha_slow: 0.0
 * /amcl/resample_interval: 1
 * /amcl/transform_tolerance: 0.5
 * /amcl/update_min_a: 0.2
 * /amcl/update_min_d: 0.2
 * /laser_filter/scan_filter_chain: [{'type': 'laser_...
 * /move_base/DWAPlannerROS/acc_lim_theta: 3.2
 * /move_base/DWAPlannerROS/acc_lim_x: 2.0
 * /move_base/DWAPlannerROS/acc_lim_y: 0.0
 * /move_base/DWAPlannerROS/controller_frequency: 10.0
 * /move_base/DWAPlannerROS/forward_point_distance: 0.325
 * /move_base/DWAPlannerROS/goal_distance_bias: 20.0
 * /move_base/DWAPlannerROS/latch_xy_goal_tolerance: False
 * /move_base/DWAPlannerROS/max_scaling_factor: 0.2
 * /move_base/DWAPlannerROS/max_vel_theta: 1.82
 * /move_base/DWAPlannerROS/max_vel_trans: 0.26
 * /move_base/DWAPlannerROS/max_vel_x: 0.26
 * /move_base/DWAPlannerROS/max_vel_y: 0.0
 * /move_base/DWAPlannerROS/min_vel_theta: 0.9
 * /move_base/DWAPlannerROS/min_vel_trans: 0.13
 * /move_base/DWAPlannerROS/min_vel_x: 0.0
 * /move_base/DWAPlannerROS/min_vel_y: 0.0
 * /move_base/DWAPlannerROS/occdist_scale: 0.02
 * /move_base/DWAPlannerROS/oscillation_reset_dist: 0.05
 * /move_base/DWAPlannerROS/path_distance_bias: 32.0
 * /move_base/DWAPlannerROS/publish_cost_grid_pc: True
 * /move_base/DWAPlannerROS/publish_traj_pc: True
 * /move_base/DWAPlannerROS/scaling_speed: 0.25
 * /move_base/DWAPlannerROS/sim_time: 2.0
 * /move_base/DWAPlannerROS/stop_time_buffer: 0.2
 * /move_base/DWAPlannerROS/vth_samples: 40
 * /move_base/DWAPlannerROS/vx_samples: 20
 * /move_base/DWAPlannerROS/vy_samples: 0
 * /move_base/DWAPlannerROS/xy_goal_tolerance: 0.05
 * /move_base/DWAPlannerROS/yaw_goal_tolerance: 0.17
 * /move_base/base_local_planner: dwa_local_planner...
 * /move_base/conservative_reset_dist: 3.0
 * /move_base/controller_frequency: 10.0
 * /move_base/controller_patience: 15.0
 * /move_base/global_costmap/cost_scaling_factor: 3.0
 * /move_base/global_costmap/footprint: [[-0.205, -0.155]...
 * /move_base/global_costmap/global_frame: map
 * /move_base/global_costmap/inflation_radius: 1.0
 * /move_base/global_costmap/map_type: costmap
 * /move_base/global_costmap/observation_sources: scan
 * /move_base/global_costmap/obstacle_range: 30.0
 * /move_base/global_costmap/plugins: [{'type': 'costma...
 * /move_base/global_costmap/publish_frequency: 10.0
 * /move_base/global_costmap/raytrace_range: 30.0
 * /move_base/global_costmap/robot_base_frame: base_footprint
 * /move_base/global_costmap/scan/clearing: True
 * /move_base/global_costmap/scan/data_type: LaserScan
 * /move_base/global_costmap/scan/marking: True
 * /move_base/global_costmap/scan/sensor_frame: base_scan
 * /move_base/global_costmap/scan/topic: scan_filtered
 * /move_base/global_costmap/static_map: True
 * /move_base/global_costmap/transform_tolerance: 0.5
 * /move_base/global_costmap/update_frequency: 10.0
 * /move_base/local_costmap/cost_scaling_factor: 3.0
 * /move_base/local_costmap/footprint: [[-0.205, -0.155]...
 * /move_base/local_costmap/global_frame: odom
 * /move_base/local_costmap/height: 3
 * /move_base/local_costmap/inflation_radius: 1.0
 * /move_base/local_costmap/map_type: costmap
 * /move_base/local_costmap/observation_sources: scan
 * /move_base/local_costmap/obstacle_range: 30.0
 * /move_base/local_costmap/publish_frequency: 10.0
 * /move_base/local_costmap/raytrace_range: 30.0
 * /move_base/local_costmap/resolution: 0.05
 * /move_base/local_costmap/robot_base_frame: base_footprint
 * /move_base/local_costmap/rolling_window: True
 * /move_base/local_costmap/scan/clearing: True
 * /move_base/local_costmap/scan/data_type: LaserScan
 * /move_base/local_costmap/scan/marking: True
 * /move_base/local_costmap/scan/sensor_frame: base_scan
 * /move_base/local_costmap/scan/topic: scan_filtered
 * /move_base/local_costmap/static_map: False
 * /move_base/local_costmap/transform_tolerance: 0.5
 * /move_base/local_costmap/update_frequency: 10.0
 * /move_base/local_costmap/width: 3
 * /move_base/oscillation_distance: 0.2
 * /move_base/oscillation_timeout: 10.0
 * /move_base/planner_frequency: 5.0
 * /move_base/planner_patience: 5.0
 * /move_base/shutdown_costmaps: False
 * /robot_description: <?xml version="1....
 * /robot_state_publisher/publish_frequency: 50.0
 * /robot_state_publisher/tf_prefix:
 * /rosdistro: melodic
 * /rosversion: 1.14.10

NODES
  /
    amcl (amcl/amcl)
    laser_filter (laser_filters/scan_to_scan_filter_chain)
    map_server (map_server/map_server)
    move_base (move_base/move_base)
    robot_state_publisher (robot_state_publisher/robot_state_publisher)
    rviz (rviz/rviz)

ROS_MASTER_URI=http://takuya-waffle-pi.local:11311

process[robot_state_publisher-1]: started with pid [25838]
process[map_server-2]: started with pid [25839]
process[amcl-3]: started with pid [25840]
process[move_base-4]: started with pid [25844]
process[rviz-5]: started with pid [25848]
process[laser_filter-6]: started with pid [25852]
[ERROR] [1608206917.974447288]: Could not parse visual element for Link [2m_frame_link]
[ERROR] [1608206917.997257723]: Failed to build tree: child link [camera_link] of joint [d435i_joint] not found
[robot_state_publisher-1] process has died [pid 25838, exit code 1, cmd /opt/ros/melodic/lib/robot_state_publisher/robot_state_publisher __name:=robot_state_publisher __log:=/home/takuya/.ros/log/2019eb2c-4054-11eb-b925-b827eb5b1dad/robot_state_publisher-1.log].
log file: /home/takuya/.ros/log/2019eb2c-4054-11eb-b925-b827eb5b1dad/robot_state_publisher-1*.log
[ERROR] [1608206919.459086315]: Could not parse visual element for Link [2m_frame_link]
[ERROR] [1608206919.459470333]: Failed to build tree: child link [camera_link] of joint [d435i_joint] not found
^C[laser_filter-6] killing on exit
[rviz-5] killing on exit
[move_base-4] killing on exit
[amcl-3] killing on exit
[map_server-2] killing on exit
shutting down processing monitor...
... shutting down processing monitor complete
done

File: urdf/waffle_pi/with_d435i/lidar-original.xacro (robot description, xacro)
@@ -161,30 +161,5 @@
     </inertial>
   </link>
-  <joint name="camera_joint" type="fixed">
-    <origin xyz="0.073 -0.011 0.084" rpy="0 0 0"/>
-    <parent link="base_link"/>
-    <child link="camera_link"/>
-  </joint>
-  <link name="camera_link">
-    <collision>
-      <origin xyz="0.005 0.011 0.013" rpy="0 0 0"/>
-      <geometry>
-        <box size="0.015 0.030 0.027"/>
-      </geometry>
-    </collision>
-  </link>
-  <joint name="camera_rgb_joint" type="fixed">
-    <origin xyz="0.003 0.011 0.009" rpy="0 0 0"/>
-    <parent link="camera_link"/>
-    <child link="camera_rgb_frame"/>
-  </joint>
-  <link name="camera_rgb_frame"/>
-  <joint name="camera_rgb_optical_joint" type="fixed">
-    <origin xyz="0 0 0" rpy="-1.57 0 -1.57"/>
-    <parent link="camera_rgb_frame"/>
-    <child link="camera_rgb_optical_frame"/>
-  </joint>
-  <link name="camera_rgb_optical_frame"/>
-  <link name="d435i_link">
+  <link name="2m_frame_link">
     <visual>
       <geometory>
@@ -195,8 +170,11 @@
     </visual>
   </link>
+  <joint name="2m_frame_joint" type="fixed">
+    <parent link="base_link"/>
+    <child link="2m_frame_link" />
+  </joint>
   <joint name="d435i_joint" type="fixed">
-    <parent link="base_link"/>
-    <child link="d435i_link" />
+    <parent link="2m_frame_link"/>
+    <child link="camera_link"/>
   </joint>
-  <xacro:sensor_d435i parent="base_link" name="d435" use_nominal_extrinsics="true"/>
 </robot>
